Commit message: First Commit
Copy of the Hydran00 directory, some settings edited in the config files

File: urdf/ur.ros2_control.xacro (robot description, xacro)
@@ -8,5 +8,5 @@
     sim_ignition:=false
     headless_mode:=false
-    initial_positions:=${dict(shoulder_pan_joint=0.0,shoulder_lift_joint=-1.57,elbow_joint=0.0,wrist_1_joint=-1.57,wrist_2_joint=0.0,wrist_3_joint=0.0)}
+    initial_positions:=${dict(shoulder_pan_joint=3.2,shoulder_lift_joint=2.4,elbow_joint=1.3,wrist_1_joint=-0.6,wrist_2_joint=3.14,wrist_3_joint=0.0)}
     use_tool_communication:=false
     hash_kinematics robot_ip

File: urdf/ur.urdf.xacro (robot description, xacro)
@@ -78,5 +78,5 @@
      script_command_port="$(arg script_command_port)"
      >
-     <origin xyz="0 0 1.79" rpy="3.14159 0 3.14159" />
+     <origin xyz="0 0 0" rpy="0 0 0" />
    </xacro:ur_robot>
    <!-- <xacro:if value="$(arg sim_gazebo)">

File: urdf/ur_macro.xacro (robot description, xacro)
@@ -62,5 +62,5 @@
     sim_ignition:=false
     headless_mode:=false
-    initial_positions:=${dict(shoulder_pan_joint=0.0,shoulder_lift_joint=-1.57,elbow_joint=0.0,wrist_1_joint=-1.57,wrist_2_joint=0.0,wrist_3_joint=0.0)}
+    initial_positions:=${dict(shoulder_pan_joint=03.2,shoulder_lift_joint=2.4,elbow_joint=1.3,wrist_1_joint=-0.6,wrist_2_joint=3.14,wrist_3_joint=0.0)}
     use_tool_communication:=false
     tool_voltage:=0
@@ -350,5 +350,5 @@
       <parent link="${prefix}wrist_3_link" />
       <child link="${prefix}flange" />
-      <origin xyz="0 0 0.1" rpy="0 ${-pi/2.0} ${-pi/2.0}" />
+      <origin xyz="0 0 0.208" rpy="0 ${-pi/2.0} ${-pi/2.0}" />
     </joint>
     <!-- ROS-Industrial 'tool0' frame - all-zeros tool frame -->
